Commit message: restructuring 1
Signed-off-by: Christoph Hellmann Santos <christoph.hellmann.santos@ipa.fraunhofer.de>

File: ur5e_cell_moveit_config/config/ur5e_workcell.ros2_control.xacro (robot description, xacro)
@@ -1,5 +1,5 @@
 <?xml version="1.0"?>
 <robot xmlns:xacro="http://www.ros.org/wiki/xacro">
-    <xacro:macro name="ur5_msa_ros2_control" params="name initial_positions_file">
+    <xacro:macro name="ur5e_workcell_ros2_control" params="name initial_positions_file">
         <xacro:property name="initial_positions" value="${load_yaml(initial_positions_file)['initial_positions']}"/>
         <ros2_control name="${name}" type="system">

File: ur5e_cell_moveit_config/config/ur5e_workcell.urdf.xacro (robot description, xacro)
@@ -12,5 +12,5 @@
     <xacro:arg name="robot_ip" default="192.168.56.2" />
     <xacro:arg name="prefix" default="" />
-    <!-- Import ur5_msa urdf file -->
+    <!-- Import ur5e_workcell urdf file -->
     <xacro:include filename="$(find ur5e_cell_description)/urdf/workcell.urdf.xacro" />
 </robot>

File: ur5e_cell_moveit_config/config/ur5e_workcell_fake.urdf.xacro (robot description, xacro)
@@ -12,5 +12,5 @@
     <xacro:arg name="robot_ip" default="192.168.56.2" />
     <xacro:arg name="prefix" default="" />
-    <!-- Import ur5_msa urdf file -->
+    <!-- Import ur5e_workcell urdf file -->
     <xacro:include filename="$(find ur5e_cell_description)/urdf/workcell.urdf.xacro" />
 </robot>
