Commit message: add camera

File: ur5e_cell_description/urdf/workcell.urdf.xacro (robot description, xacro)
@@ -5,4 +5,5 @@
     <xacro:include filename="$(find ur5e_cell_description)/urdf/robot_cell.xacro" />
     <xacro:include filename="$(find ur_description)/urdf/ur_macro.xacro" />
+    <xacro:include filename="$(find realsense2_description)/urdf/_d435.urdf.xacro" />
     <xacro:property name="gripper_name" value="shunk_egp50" />
     <xacro:property name="initial_positions_file" default="$(find ur5e_cell_description)/config/initial_positions.yaml" />
@@ -39,4 +40,8 @@
     <xacro:arg name="initial_positions_file" default="$(find ur5e_cell_description)/config/initial_positions.yaml" />
     <xacro:arg name="use_nominal_extrinsics" default="false" />
+    <xacro:arg name="add_plug" default="false" />
+    <xacro:arg name="use_mesh" default="true" />
+    <!-- Args related to realsense -->
+    <xacro:arg name="use_nominal_extrinsics" default="false"/>
     <xacro:arg name="add_plug" default="false" />
     <xacro:arg name="use_mesh" default="true" />
@@ -96,3 +101,6 @@
         <origin xyz="0.0 0.0 0.0" rpy="0.0 0.0 0.0" />
     </joint>
+    <xacro:sensor_d435 parent="tool0" use_nominal_extrinsics="$(arg use_nominal_extrinsics)"  add_plug="$(arg add_plug)" use_mesh="$(arg use_mesh)">
+        <origin xyz="0 -0.05 0" rpy="${pi/2} ${pi/2} 0"/>
+    </xacro:sensor_d435>
 </robot>
